File: hardware/pcb/mosfet/mosfet_smt_test.brd (EAGLE design)
At the start: 58.4 x 88.6 mm, 45 parts, among them J10 M2_CTRL_IN_TEST, J11 M3_CTRL_IN_TEST, J12 M4_CTRL_IN_TEST, J13 GND_TEST, J14 M3_DRAIN_TEST, J16 M4_DRAIN_TEST, J20 M2_DRAIN_TEST, J23 M1_DRAIN_TEST, J8 VIN_TEST, J9 M1_CTRL_IN_TEST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

Commit message: finalized circuit boards and ordered w/ gerber files
Other:
- board text added: "C:/Users/cbaro/OneDrive/Pictures/picodrone.bmp"
